Commit message: Added refined xacro model for WSG 50 gripper

File: wsg_50_simulation/urdf/wsg_50.urdf.xacro (robot description, xacro)
@@ -3,10 +3,10 @@
 	xmlns:controller="http://playerstage.sourceforge.net/gazebo/xmlschema/#controller"
 	xmlns:interface="http://playerstage.sourceforge.net/gazebo/xmlschema/#interface"
-        xmlns:xacro="http://ros.org/wiki/xacro"
+    xmlns:xacro="http://ros.org/wiki/xacro"
 	name="wsg_50">
 <!-- finger_length: Length of finger from gripper base. (was 0.023) -->
 <!-- finger_tip:    Offset of finger tip along fingers' motion direction.
                     Use e.g. for single contact point tip on finger. (default 0) -->
-<xacro:macro name="wsg_50_xacro" params="name parent finger_length finger_tip *origin">
+<xacro:macro name="wsg_50_xacro" params="name parent finger_length finger_tip off_dist rotation *origin">
  <joint name="${name}_anterior_gripper_joint" type="fixed">
     <insert_block name="origin"/>
@@ -18,5 +18,5 @@
       <inertial>
           <mass value="0.25" />
-          <origin xyz="0 0 0" />
+          <origin xyz="0.0 0.0 ${off_dist}" rpy="0.0 0.0 ${rotation}" />
      	  <!--inertia ixx="1.0" ixy="0.0" ixz="0.0"
                iyy="100.0" iyz="0.0"
@@ -25,5 +25,5 @@
       </inertial>
       <visual>
-          <origin xyz="0.0 0 0" rpy="0 0 0" />
+          <origin xyz="0.0 0.0 ${off_dist}" rpy="0 0 ${rotation}" />
           <geometry>
              <mesh filename="package://wsg_50_simulation/meshes/WSG50_110.stl" scale="1 1 1"/>
@@ -35,5 +35,5 @@
       </visual>
       <collision>
-          <origin xyz="0.0 0 0" rpy="0 0 0" />
+          <origin xyz="0.0 0.0 ${off_dist}" rpy="0 0 ${rotation}" />
           <geometry>
 	     <!--box size="0.146 0.05 0.0735"/-->
@@ -56,5 +56,5 @@
   <joint name="${name}_finger_left_joint" type="prismatic">
      <limit lower="-0.055" upper="-0.0027" effort="1.0" velocity="1.0"/>
-     <origin xyz="0 0 0" rpy="0 0 0" />      <!--origin xyz="-0.0067 0 0.049" rpy="0 0 0" /-->
+     <origin xyz="0 0 0" rpy="0 0 ${rotation}" />      <!--origin xyz="-0.0067 0 0.049" rpy="0 0 0" /-->
      <parent link="${name}_base_link"/>
      <child link="${name}_gripper_left" />
@@ -141,5 +141,5 @@
   <joint name="${name}_finger_right_joint" type="prismatic">
      <limit lower="0.0027" upper="0.055" effort="1.0" velocity="1.0"/>
-     <origin xyz="0 0 0" rpy="0 0 3.14159" />
+     <origin xyz="0 0 0" rpy="0 0 -${rotation}" />
      <parent link="${name}_base_link"/>
      <child link="${name}_gripper_right" />
